File: Hardware/NewtonCart.kicad_pcb (KiCad board)
At the start: 2 copper layers, 18 parts, among them J1 Battery Pins, J10 LOADCELL, J2 TP4056 Module, J3 Reserve IO's, J4 UART2TTL Bridge, J5 BoostConverter, J6 MPU6050, J7 HX711, J8 HC-SR04, J9 FOTOELECTRIC_ENCODER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

Commit message: Cambios Placa al 190322
Parts:
- moved J5 16.3 mm to (94.0, 143.5), turned to -90 degrees
- moved J9 9.53 mm to (120.0, 126.4)
- moved C2 8.92 mm to (95.9, 147.3)
- moved J10 8.04 mm to (71.1, 125.7)
- moved J1 8.03 mm to (57.1, 125.7)
- moved R1 7.73 mm to (124.5, 141.0)
- moved C1 6.87 mm to (95.9, 144.8), turned to 0 degrees
- moved J8 6.84 mm to (71.1, 138.4)
- moved U1 6.48 mm to (137.2, 134.0)
- moved J3 6.48 mm to (149.9, 127.0)
- moved R4 6.48 mm to (149.9, 135.9)
- moved J2 6.48 mm to (52.1, 137.7)
- moved J7 6.48 mm to (82.9, 121.4)
- moved J6 6.02 mm to (123.7, 144.1)
- moved J4 5.72 mm to (137.2, 156.8)
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Connections:
- C1 pad 2: Battery(-) -> 4056OUT-
- C2 pad 2: Battery(-) -> 4056OUT-
- J1 pad 3: Battery(-) -> 4056OUT-
- J1 pad 4: Battery(-) -> 4056OUT-
- J2 pad 2: Battery(-) -> 4056OUT-
- J2 pad 5: Battery(-) -> 4056OUT-
- J2 pad 6: Battery(-) -> 4056OUT-
- J3 pad 1: Net-(J3-Pad1) -> Net-(U1-Pad9)
- J3 pad 2: Net-(J3-Pad2) -> Net-(U1-Pad8)
- J4 pad 1: Battery(-) -> 4056OUT-
- J5 pad 2: Battery(-) -> 4056OUT-
- J5 pad 4: Battery(-) -> 4056OUT-
- J6 pad 2: MPU_SDA -> 4056OUT-
- J6 pad 4: Battery(-) -> MPU_SDA
- J7 pad 6: Battery(-) -> 4056OUT-
- J8 pad 4: Battery(-) -> 4056OUT-
- J9 pad 3: Battery(-) -> 4056OUT-
- R1 pad 1: Battery(-) -> 4056OUT-
- R2 pad 1: Battery(-) -> 4056OUT-
- U1 pad 1: Battery(-) -> 4056OUT-
- U1 pad 15: Battery(-) -> 4056OUT-
- U1 pad 30: LC_SCK -> LC_DT
- U1 pad 31: LC_DT -> LC_SCK
- U1 pad 38: Battery(-) -> 4056OUT-
- U1 pad 39: Battery(-) -> 4056OUT-
- U1 pad 6: Net-(J3-Pad3) -> VEL_PULSE
- U1 pad 7: VEL_PULSE -> Net-(J3-Pad3)
- U1 pad 8: Net-(J3-Pad1) -> Net-(U1-Pad8)
- U1 pad 9: Net-(J3-Pad2) -> Net-(U1-Pad9)
- U2 pad 1: Battery(-) -> 4056OUT-
Routing:
- net 4056OUT-: track 0.00 -> 232.4 mm
- net 3.3Reg: track 0.00 -> 96.4 mm
- net US_TRIGGER: track 0.00 -> 83.9 mm
- net Boost5V: track 0.00 -> 81.2 mm
- net Battery(+): track 0.00 -> 39.9 mm
- net LC_A-: track 0.00 -> 28.4 mm
- net Net-(J4-Pad2): track 0.00 -> 27.7 mm
- net LC_A+: track 0.00 -> 24.8 mm
- net VEL_PULSE: track 0.00 -> 21.9 mm
- net LC_E-: track 0.00 -> 21.4 mm
- net LC_DT: track 0.00 -> 17.8 mm
- net LC_SCK: track 0.00 -> 17.3 mm
- net Net-(J8-Pad3): track 0.00 -> 17.1 mm
- net 4056OUT+: track 0.00 -> 16.9 mm
- net LC_E+: track 0.00 -> 16.9 mm
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